File: AN6291_encoder/AN6291_encoder.kicad_sch (KiCad schematic)
At the start: 130 parts, among them IC1 TPS70960DBVT, J1 input mic, J2 output, J3 batt, J4 input line, Q1 NPN, Q2 NPN, Q3 BC848, Q4 BCV62, Q5 BCV62, Q6 BC848, U3 OPA1612AxD, U4 OPA1612AxD

Commit message: Removed voltage regulator for microphone supply now powered from 9v battery for lower noise
Parts:
- removed IC1: TPS70960DBVT, LIB_TPS70960DBVT:SOT95P280X145-5N, symbol TPS70960DBVT:TPS70960DBVT
- added R37: 100R, Resistor_SMD:R_0805_2012Metric, symbol Device:R_Small
- C24, C30: footprint Capacitor_SMD:C_0805_2012Metric -> Capacitor_SMD:C_1206_3216Metric
Connections:
- net VCC: now also R37.1
- net +6V renamed 9V mic
- net 9V mic: now also R37.2
Other:
- moved on the sheet: C36

Commit message: rev B
Parts:
- C1, C14, C15, C16, C17, C18, C19, C2, C21, C23, C24, C25, C26, C28, C3, C30, C31, C32, C33, C34, C35, C36, C37, C38, C39, C4, C40, C41, C42, C43, C44, C45, C46, C47, C5, C50, C6, C7, C8, C9, F1, J1, J2, J3, J4, Q1, Q2, Q3, Q4, Q5, Q6, RV1, S1, TP1, TP3, U1, U3, U4: now left out of the parts list
- C10, C11, C12, C13: value 100n -> 100nf; now left out of the parts list
- C20, C22: value 10nf COG -> 10nf; now left out of the parts list
- C27, C29: value 0.1uf -> 100nf; now left out of the parts list
- R1, R19, R2: JLCPCB Part (none) -> C17513
- R10, R13, R15, R7: JLCPCB Part (none) -> C17633
- R11, R9: JLCPCB Part (none) -> C17470
- R12, R5: JLCPCB Part (none) -> C17589
- R14, R8: JLCPCB Part (none) -> C17673
- R16: JLCPCB Part (none) -> C17772; JLCPCB Part  (none) -> C17772
- R17, R4: JLCPCB Part (none) -> C26010
- R18, R3: JLCPCB Part (none) -> C17414
- R20, R21: JLCPCB Part (none) -> C28636
- R22, R29: JLCPCB Part (none) -> C17630
- R23, R26, R27, R32: JLCPCB Part (none) -> C17475
- R24, R31: JLCPCB Part (none) -> C17737; now left out of the parts list
- R25, R28: JLCPCB Part (none) -> C17737
- R30, R38: JLCPCB Part (none) -> C17560
- R33, R35, R40, R42: value 274R -> 270R; JLCPCB Part (none) -> C17590
- R34, R39: value 57,6K -> 56k; JLCPCB Part (none) -> C17756
- R36, R41: JLCPCB Part (none) -> C17604
- R37, R60, R61: JLCPCB Part (none) -> C17408
- R48, R49, R58, R59: value 100 -> 100R; JLCPCB Part (none) -> C17408
- R50, R53: value 4.1k -> 4.7k; JLCPCB Part (none) -> C17673
- R51, R52, R62, R63: JLCPCB Part (none) -> C149504
- R54, R55, R56, R57: JLCPCB Part (none) -> C17539
- R6: JLCPCB Part (none) -> C17772
- R64, R65: JLCPCB Part (none) -> C17513; now left out of the parts list
